Commit message: big track aand better void

File: resources/plane.urdf (robot description, URDF)
Before this commit: robot plane, 1 links, 0 joints
Links:
- link base_link: geometry collision box size=40 40 0.01; visual box size=40 40 0.01

Commit message: made proper track

File: resources/plane.urdf (robot description, URDF)
Before this commit: robot plane, 1 links, 0 joints
Links:
- link base_link: geometry collision box size=100 100 0.01; visual box size=100 100 0.01

Commit message: more changes to update old gym

File: resources/plane.urdf (robot description, URDF)
Before this commit: robot plane, 1 links, 0 joints
Links:
- link base_link: geometry collision box size=150 150 1; visual box size=150 150 1
