Commit message: #wigglywobblynomore

File: resources/car.urdf (robot description, URDF)
Before this commit: robot car, 7 links, 6 joints
Links:
- link base_link: mass 6 -> 400
- link left_back_wheel: mass 0.3 -> 115
- link left_front_wheel: mass 0.3 -> 95
- link left_hinge: mass 0.01 -> 20
- link right_back_wheel: mass 0.3 -> 115
- link right_front_wheel: mass 0.3 -> 95
- link right_hinge: mass 0.01 -> 20
Joints:
- joint base_to_left_back_wheel: origin xyz=-0.2 0.175 0 -> xyz=-0.2 0.175 0 rpy=0 0 0
- joint base_to_right_back_wheel: origin xyz=-0.2 -0.175 0 -> xyz=-0.2 -0.175 0 rpy=0 0 0
- joint left_hinge_to_left_front_wheel: origin xyz=0 0.2 0 -> xyz=0 0.15 0 rpy=0 0 0
- joint right_hinge_to_right_front_wheel: origin xyz=0 -0.2 0 -> xyz=0 -0.15 0 rpy=0 0 0
